File: pcb/RH020.1/RH020.1.brd (EAGLE design)
At the start: 49.5 x 49.5 mm, 28 parts, among them CN1 USB, CN4 FTDI, U2 FT232RLSSOP, U3 REG1117

Commit message: updated pcb design and gerbers
Other:
- board text added: "RH020.1 Nov 2015"
- board text added: "Wifi 7 Segment smd Richard Hawthorn richardhawthorn.com"
- board text removed: "RH018.2 Nov 2015"
- board text removed: "Wifi 7 Segment Richard Hawthorn richardhawthorn.com"
Changed lines of the file:
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@@
 <wire x1="3.175" y1="49.53" x2="46.355" y2="49.53" width="0.0254" layer="20"/>
 <wire x1="49.53" y1="46.355" x2="49.53" y2="3.175" width="0.0254" layer="20"/>
-<text x="1.27" y="7.0485" size="1.016" layer="25">RH018.2
+<text x="1.27" y="7.0485" size="1.016" layer="25">RH020.1
 Nov 2015</text>
-<text x="25.4" y="0.3175" size="1.016" layer="25">Wifi 7 Segment
+<text x="25.4" y="0.3175" size="1.016" layer="25">Wifi 7 Segment smd
 Richard Hawthorn
 richardhawthorn.com</text>
