File: pcb/RH020.1/RH020.1.sch (EAGLE design)
At the start: 27 parts, among them CN1 USB, CN4 FTDI, U2 FT232RLSSOP, U3 REG1117

Commit message: updated pcb design and gerbers
Other:
- note added: "Wifi 7 Segment"
- note removed: "7 Segment Node"
Changed lines of the file:
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@@
 <sheet>
 <plain>
-<text x="166.116" y="15.748" size="3.81" layer="94" font="vector" ratio="10">7 Segment Node</text>
+<text x="166.116" y="15.748" size="3.81" layer="94" font="vector" ratio="10">Wifi 7 Segment </text>
 <text x="217.678" y="20.32" size="2.1844" layer="94" font="vector">richardhawthorn.com</text>
 <text x="166.37" y="8.382" size="2.54" layer="94" font="vector">Richard Hawthorn</text>
